Commit message: Added two transmissions

File: urdf/m1.xacro (robot description, xacro)
@@ -39,4 +39,14 @@
     <axis xyz="0 0 1" />
   </joint>
+  <transmission name="left_wheel">
+    <type>transmission_interface/SimpleTransmission</type>
+    <joint name="base_to_lwheel">
+      <hardwareInterface>VelocityJointInterface</hardwareInterface>
+    </joint>
+    <actuator name="left_motor">
+      <hardwareInterface>VelocityJointInterface</hardwareInterface>
+      <mechanicalReduction>1</mechanicalReduction>
+    </actuator>
+  </transmission>
   <link name="rwheel">
     <visual>
@@ -54,4 +64,14 @@
     <axis xyz="0 0 1" />
   </joint>
+  <transmission name="right_wheel">
+    <type>transmission_interface/SimpleTransmission</type>
+    <joint name="base_to_rwheel">
+      <hardwareInterface>VelocityJointInterface</hardwareInterface>
+    </joint>
+    <actuator name="right_motor">
+      <hardwareInterface>VelocityJointInterface</hardwareInterface>
+      <mechanicalReduction>1</mechanicalReduction>
+    </actuator>
+  </transmission>
   <link name="fwheel_attach">
     <visual>

Commit message: Snapshot

File: urdf/m1.xacro (robot description, xacro)
@@ -1,4 +1,4 @@
 <?xml version="1.0"?>
-<robot xmlns:xacro="http://www.ros.org/wiki/xacro" name="m1">
+<robot xmlns:xacro="http://www.ros.org/wiki/xacro" name="mmm_bot">
   <xacro:property name="body_length" value="0.6096" />>
   <xacro:property name="body_width" value="0.3048" />
@@ -7,4 +7,11 @@
   <xacro:property name="wheel_spacer" value="0.00635" />>
   <xacro:property name="wheel_width" value="0.040" />
+  <!--xacro:include filename="$(find m1)/robots/m1.gazebo" /-->
+  <gazebo>
+    <plugin name="gazebo_ros_control" filename="libgazebo_ros_control.so">
+      <robotNamespace>mmm_bot</robotNamespace>
+      <robotSimType>gazebo_ros_control/DefaultRobotHWSim</robotSimType>
+    </plugin>
+  </gazebo>
   <!-- Materials -->
   <material name="base">
@@ -23,4 +30,12 @@
       <material name="base" />
     </visual>
+    <inertial>
+        <origin xyz="0 0 0" rpy="0 0 0" />
+        <mass value="1" />
+        <inertia
+          ixx="1.0" ixy="0.0" ixz="0.0"
+          iyy="1.0" iyz="0.0"
+          izz="1.0" />
+    </inertial>
   </link>
   <link name="lwheel">
@@ -32,4 +47,12 @@
       <material name="wheel" />
     </visual>
+    <inertial>
+        <origin xyz="0 0 0" rpy="0 0 0" />
+        <mass value="1" />
+        <inertia
+          ixx="1.0" ixy="0.0" ixz="0.0"
+          iyy="1.0" iyz="0.0"
+          izz="1.0" />
+    </inertial>
   </link>
   <joint name="base_to_lwheel" type="continuous">
@@ -42,8 +65,8 @@
     <type>transmission_interface/SimpleTransmission</type>
     <joint name="base_to_lwheel">
-      <hardwareInterface>VelocityJointInterface</hardwareInterface>
+      <hardwareInterface>hardware_interface/VelocityJointInterface</hardwareInterface>
     </joint>
     <actuator name="left_motor">
-      <hardwareInterface>VelocityJointInterface</hardwareInterface>
+      <hardwareInterface>hardware_interface/VelocityJointInterface</hardwareInterface>
       <mechanicalReduction>1</mechanicalReduction>
     </actuator>
@@ -57,4 +80,12 @@
       <material name="wheel" />
     </visual>
+    <inertial>
+        <origin xyz="0 0 0" rpy="0 0 0" />
+        <mass value="1" />
+        <inertia
+          ixx="1.0" ixy="0.0" ixz="0.0"
+          iyy="1.0" iyz="0.0"
+          izz="1.0" />
+    </inertial>
   </link>
   <joint name="base_to_rwheel" type="continuous">
@@ -67,8 +98,8 @@
     <type>transmission_interface/SimpleTransmission</type>
     <joint name="base_to_rwheel">
-      <hardwareInterface>VelocityJointInterface</hardwareInterface>
+      <hardwareInterface>hardware_interface/VelocityJointInterface</hardwareInterface>
     </joint>
     <actuator name="right_motor">
-      <hardwareInterface>VelocityJointInterface</hardwareInterface>
+      <hardwareInterface>hardware_interface/VelocityJointInterface</hardwareInterface>
       <mechanicalReduction>1</mechanicalReduction>
     </actuator>
@@ -84,4 +115,12 @@
       </material>
     </visual>
+    <inertial>
+        <origin xyz="0 0 0" rpy="0 0 0" />
+        <mass value="1" />
+        <inertia
+          ixx="1.0" ixy="0.0" ixz="0.0"
+          iyy="1.0" iyz="0.0"
+          izz="1.0" />
+    </inertial>
   </link>
   <joint name="base_to_fattach" type="fixed">
@@ -98,4 +137,12 @@
       <material name="wheel" />
     </visual>
+    <inertial>
+        <origin xyz="0 0 0" rpy="0 0 0" />
+        <mass value="1" />
+        <inertia
+          ixx="1.0" ixy="0.0" ixz="0.0"
+          iyy="1.0" iyz="0.0"
+          izz="1.0" />
+    </inertial>
   </link>
   <joint name="base_to_fwheel" type="continuous">
@@ -115,4 +162,12 @@
       </material>
     </visual>
+    <inertial>
+        <origin xyz="0 0 0" rpy="0 0 0" />
+        <mass value="1" />
+        <inertia
+          ixx="1.0" ixy="0.0" ixz="0.0"
+          iyy="1.0" iyz="0.0"
+          izz="1.0" />
+    </inertial>
   </link>
   <joint name="base_to_scanner" type="fixed">
